File: test_boards/10CL006/10CL006.kicad_pcb (KiCad board)
At the start: 2 copper layers, 75 parts, among them IC1 10CL006YE144C8G, J1 CL_JTAG, U1 W25Q128JVS, Y1 SG-7050CAN

Commit message: Добавлен полный тест API
Parts:
- C10, C11, C12, C13, C14, C19, C20, C21, C22, C23, C24, C25, C26, C27, C28, C29, C30, C31, C32, C33, C34, C35, C36, C37, C38, C39, C40, C41, C42, C43, C44, C45, C5, C50, C51, C52, C53, C6, C7, C8, C9: moved to B.Cu
- moved IC1 60.2 mm to (144.4, 80.7)
- moved C13 40.0 mm to (138.2, 73.3), turned to -90 degrees
- moved C10 22.0 mm to (122.2, 66.0), turned to 180 degrees
- moved C11 22.0 mm to (122.2, 68.0), turned to 180 degrees
- moved C12 22.0 mm to (122.2, 69.9), turned to 180 degrees
- moved C5 22.0 mm to (122.2, 56.1), turned to 180 degrees
- moved C6 22.0 mm to (122.2, 58.1), turned to 180 degrees
- moved C7 22.0 mm to (122.2, 60.1), turned to 180 degrees
- moved C8 22.0 mm to (122.2, 62.0), turned to 180 degrees
- moved C9 22.0 mm to (122.2, 64.0), turned to 180 degrees
- moved C14 22.0 mm to (125.4, 58.1), turned to 180 degrees
- turned C19 to 180 degrees
- turned C20 to 180 degrees
- turned C21 to 180 degrees
- turned C22 to 180 degrees
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Routing:
- net +3V3_VCCIO: track 0.00 -> 2.76 mm, vias 0 -> 1
