File: test_boards/10CL006YE144C8G/10CL006YE144C8G.kicad_sch (KiCad schematic)
At the start: 75 parts, among them IC1 10CL006YE144C8G, J1 CL_JTAG, U1 W25Q128JVS, Y1 SG-7050CAN

Commit message: Обновлён файл KiCad проекта
Parts:
- removed C1, C2, C3, C4, C46, C47, C48, C49, C54, C56, C57, C60: 1uF, Capacitor_SMD:C_0603_1608Metric_Pad1.08x0.95mm_HandSolder, symbol Device:C
- removed C10, C11, C12, C13, C14, C15, C16, C17, C18, C19, C20, C21, C22, C23, C24, C25, C26, C28, C29, C37, C38, C5, C55, C58, C59, C6, C61, C7, C8, C9: 100 nF, Capacitor_SMD:C_0402_1005Metric_Pad0.74x0.62mm_HandSolder, symbol Device:C
- removed C27, C30, C31, C32, C33, C34, C35, C36, C39, C40, C41, C42, C43, C44, C45, C50, C51, C52, C53: 4.7 uF, Capacitor_SMD:C_0603_1608Metric_Pad1.08x0.95mm_HandSolder, symbol Device:C
- removed FB1, FB2, FB3, FB4: BLM15PD121SN1D, Inductor_SMD:L_0402_1005Metric, symbol Custom_FerriteBead:BLM15PD121SN1D
- removed IC1: 10CL006YE144C8G, Custom_Altera_FPGA:QFP50P2200X2200X165-145N, symbol Custom_Altera_FPGA:10CL006YE144C8G
- removed J1: CL_JTAG, Connector_IDC:IDC-Header_2x05_P2.54mm_Vertical, symbol Connector_Generic:Conn_02x05_Odd_Even
- removed R1: 1K, Resistor_SMD:R_0402_1005Metric_Pad0.72x0.64mm_HandSolder, symbol Device:R
- removed R2: 33, Resistor_SMD:R_0402_1005Metric_Pad0.72x0.64mm_HandSolder, symbol Device:R
- removed R3, R4, R5, R6: 2R2, Resistor_SMD:R_0402_1005Metric_Pad0.72x0.64mm_HandSolder, symbol Device:R
- removed U1: W25Q128JVS, Package_SO:SOIC-8_5.3x5.3mm_P1.27mm, symbol Memory_Flash:W25Q128JVS
- removed Y1: SG-7050CAN, Oscillator:Oscillator_SMD_SeikoEpson_SG8002CA-4Pin_7.0x5.0mm, symbol Oscillator:SG-7050CAN
- added C401, C402, C403, C404, C435, C436, C437, C438, C439, C440, C443, C444: 1uF, Capacitor_SMD:C_0603_1608Metric_Pad1.08x0.95mm_HandSolder, symbol Device:C
- added C405, C406, C407, C408, C409, C410, C411, C412, C417, C418, C419, C420, C421, C422, C423, C424, C425, C426, C427, C429, C430, C432, C433, C434, C441, C442, C445, C446, C458, C461: 100 nF, Capacitor_SMD:C_0402_1005Metric_Pad0.74x0.62mm_HandSolder, symbol Device:C
- added C413, C414, C415, C416, C428, C431, C447, C448, C449, C450, C451, C452, C453, C454, C455, C456, C457, C459, C460: 4.7 uF, Capacitor_SMD:C_0603_1608Metric_Pad1.08x0.95mm_HandSolder, symbol Device:C
- added FB401, FB402, FB403, FB404: BLM15PD121SN1D, Inductor_SMD:L_0402_1005Metric, symbol Custom_FerriteBead:BLM15PD121SN1D
- added IC401: 10CL006YE144C8G, Custom_Altera_FPGA:QFP50P2200X2200X165-145N, symbol Custom_Altera_FPGA:10CL006YE144C8G
- added J401: CL_JTAG, Connector_IDC:IDC-Header_2x05_P2.54mm_Vertical, symbol Connector_Generic:Conn_02x05_Odd_Even
- added R401: 33, Resistor_SMD:R_0402_1005Metric_Pad0.72x0.64mm_HandSolder, symbol Device:R
- added R402, R403, R408, R409: 2R2, Resistor_SMD:R_0402_1005Metric_Pad0.72x0.64mm_HandSolder, symbol Device:R
- added R404: 1K, Resistor_SMD:R_0402_1005Metric_Pad0.72x0.64mm_HandSolder, symbol Device:R
- added R407, R413, R414: 4.7K, Resistor_SMD:R_0402_1005Metric_Pad0.72x0.64mm_HandSolder, symbol Device:R
- added R410, R411, R412: 10K, Resistor_SMD:R_0402_1005Metric_Pad0.72x0.64mm_HandSolder, symbol Device:R
- added U401: W25Q128JVS, Package_SO:SOIC-8_5.3x5.3mm_P1.27mm, symbol Memory_Flash:W25Q128JVS
- added Y401: SG-7050CAN, Oscillator:Oscillator_SMD_SeikoEpson_SG8002CA-4Pin_7.0x5.0mm, symbol Oscillator:SG-7050CAN
Connections:
- net +1V2: now also C401.1, C402.1, C417.1, C418.1, FB401.1, FB402.1
- net +1V2_VCCD_PLL: now also C433.1, C434.1, C436.1, C459.1, C460.1, FB402.2, IC401.109 (VCCD_PLL2), IC401.37 (VCCD_PLL1)
- net +1V2_VCCINT: now also C415.1, C421.1, C422.1, C423.1, C424.1, C425.1, C426.1, C427.1, C428.1, C431.1, C435.1, C447.1, C448.1, C450.1, C451.1, C455.1, C458.1, FB401.2, IC401.102 (VCCINT_6), IC401.116 (VCCINT_7), IC401.134 (VCCINT_8), IC401.29 (VCCINT_2), IC401.45 (VCCINT_3), IC401.5 (VCCINT_1), IC401.61 (VCCINT_4), IC401.78 (VCCINT_5)
- net +2V5: now also C403.1, C419.1, FB403.1
- net +2V5_VCCA: now also C429.1, C430.1, C437.1, C454.1, C457.1, FB403.2, IC401.107 (VCCA2), IC401.35 (VCCA1), IC401.96 (MSEL1)
- net +3V3: now also C404.1, C420.1, C439.1, C440.1, C441.1, C442.1, FB404.1, R408.1, R409.1
- net +3V3_FLASH: now also C443.1, C445.2, R402.2, R403.2, R408.2, U401.8 (VCC)
- net +3V3_OSCILL: now also C444.1, C446.2, R404.1, R409.2, Y401.4 (VCC)
- net +3V3_VCCIO: now also C405.1, C406.1, C407.1, C408.1, C409.1, C410.1, C411.1, C412.1, C413.1, C414.1, C416.1, C432.1, C438.1, C449.1, C452.1, C453.1, C456.1, C461.1, FB404.2, IC401.117 (VCCIO7_1), IC401.122 (VCCIO7_2), IC401.130 (VCCIO8_1), IC401.139 (VCCIO8_2), IC401.17 (VCCIO1), IC401.26 (VCCIO2), IC401.40 (VCCIO3_1), IC401.47 (VCCIO3_2), IC401.56 (VCCIO4_1), IC401.62 (VCCIO4_2), IC401.81 (VCCIO5), IC401.93 (VCCIO6), J401.4 (Pin_4), R410.2, R411.2, R412.2, R413.2, R414.2
- net CL_ASDO: now also IC401.6 (IO_4), U401.5 (DI/IO_{0})
- net CL_CLK_0: now also R401.1, Y401.3 (OUT)
- net CL_CLK_0_IN: now also IC401.22 (CLK0), R401.2
- net CL_CLK_ON: now also R404.2, Y401.1 (~{ST})
- net CL_CONFIG_DONE: now also IC401.92 (CONF_DONE), R410.1
- net CL_DATA0: now also IC401.13 (IO_10), U401.2 (DO/IO_{1})
- net CL_DCLK: now also IC401.12 (IO_9), U401.6 (CLK)
- net CL_NCONFIG: now also IC401.14 (NCONFIG), R412.1
- net CL_NCSO: now also IC401.8 (IO_6), U401.1 (~{CS})
- net CL_NSTATUS: now also IC401.9 (NSTATUS), R411.1
- net CL_TCK: now also IC401.16 (TCK), J401.1 (Pin_1), R407.1
- net CL_TDI: now also IC401.15 (TDI), J401.9 (Pin_9), R414.1
- net CL_TDO: now also IC401.20 (TDO), J401.3 (Pin_3)
- net CL_TMS: now also IC401.18 (TMS), J401.5 (Pin_5), R413.1
- net FL_HOLD: now also R402.1, U401.7 (~{HOLD}/~{RESET}/IO_{3})
- net FL_WP: now also R403.1, U401.3 (~{WP}/IO_{2})
- net GND: now also C401.2, C402.2, C403.2, C404.2, C405.2, C406.2, C407.2, C408.2, C409.2, C410.2, C411.2, C412.2, C413.2, C414.2, C415.2, C416.2, C417.2, C418.2, C419.2, C420.2, C421.2, C422.2, C423.2, C424.2, C425.2, C426.2, C427.2, C428.2, C429.2, C430.2, C431.2, C432.2, C433.2, C434.2, C435.2, C436.2, C437.2, C438.2, C439.2, C440.2, C441.2, C442.2, C443.2, C444.2, C445.1, C446.1, C447.2, C448.2, C449.2, C450.2, C451.2, C452.2, C453.2, C454.2, C455.2, C456.2, C457.2, C458.2, C459.2, C460.2, C461.2, IC401.104 (GND_13), IC401.108 (GNDA2), IC401.110 (GND_14), IC401.118 (GND_15), IC401.123 (GND_16), IC401.131 (GND_17), IC401.140 (GND_18), IC401.145 (EP_(GND)), IC401.19 (GND_2), IC401.21 (NCE), IC401.27 (GND_3), IC401.30 (GND_4), IC401.36 (GNDA1), IC401.4 (GND_1), IC401.41 (GND_5), IC401.48 (GND_6), IC401.57 (GND_7), IC401.63 (GND_8), IC401.64 (GND_9), IC401.79 (GND_10), IC401.82 (GND_11), IC401.94 (MSEL0), IC401.95 (GND_12), IC401.97 (MSEL2), J401.10 (Pin_10), J401.2 (Pin_2), R407.2, U401.4 (GND), Y401.2 (GND)

Commit message: Исправлена схема платы. Добавлен конфиг 10CL006.yaml
Parts:
- renumbered C401 to C1, C410 to C10, C411 to C11, C412 to C12, C432 to C13, C461 to C14, C417 to C15, C418 to C16, C419 to C17, C420 to C18, C421 to C19, C402 to C2, C422 to C20, C423 to C21, C424 to C22, C425 to C23, C426 to C24, C427 to C25, C458 to C26, C455 to C27, C429 to C28, C430 to C29, C403 to C3, C414 to C30, C413 to C31, C452 to C32, C416 to C33, C449 to C34, C453 to C35, C456 to C36, C433 to C37, C434 to C38, C415 to C39, C404 to C4, C431 to C40, C428 to C41, C447 to C42, C448 to C43, C450 to C44, C451 to C45, C435 to C46, C436 to C47, C437 to C48, C438 to C49, C405 to C5, C454 to C50, C457 to C51, C459 to C52, C460 to C53, C440 to C54, C442 to C55, C444 to C56, C439 to C57, C446 to C58, C441 to C59, C406 to C6, C443 to C60, C445 to C61, C407 to C7, C408 to C8, C409 to C9, FB401 to FB1, FB402 to FB2, FB403 to FB3, FB404 to FB4, IC401 to IC1, J401 to J1, R404 to R1, R412 to R10, R413 to R11, R414 to R12, R407 to R2, R401 to R3, R402 to R4, R409 to R5, R403 to R6, R408 to R7, R410 to R8, R411 to R9, U401 to U1, Y401 to Y1
